Commit message: Renamed angle joint to motor joint

File: src/qube_description/urdf/qube.macro.xacro (robot description, xacro)
@@ -55,6 +55,6 @@
       <origin xyz="0 0 ${box_size/2}"/>
     </joint>
-    <!-- Angle joint -->
-    <joint name="${prefix}angle" type="revolute">
+    <!-- Motor joint -->
+    <joint name="${prefix}motor_joint" type="revolute">
       <parent link="${prefix}stator_link"/>
       <child link="${prefix}rotor_link"/>

Commit message: macroxacro

File: src/qube_description/urdf/qube.macro.xacro (robot description, xacro)
@@ -60,5 +60,5 @@
       <child link="${prefix}rotor_link"/>
       <origin xyz="0 0 ${box_size/2}"/>
-      <axis xyz="0 0 1"/>
+      <axis xyz="0 0 -1"/>
       <limit lower="-3.14159" upper="3.14159" effort="1.0" velocity="1.0"/>
     </joint>
